Commit message: URDF update

File: description/robot_frame.xacro (robot description, xacro)
@@ -1,4 +1,5 @@
 <?xml version="1.0"?>
 <robot xmlns:xacro="http://www.ros.org/wiki/xacro">
+    <!-- MATERIALS -->
     <material name="white">
         <color rgba="1 1 1 1" />
@@ -7,6 +8,9 @@
         <color rgba="0 0 0 1" />
     </material>
+    <material name="phone">
+        <color rgba="0 0 0 0.75" />
+    </material>
     <material name="blue">
-        <color rgba="0.2 0.2 1 1" />
+        <color rgba="0.0156 0.23137 0.3607 1" />
     </material>
     <material name="orange">
@@ -15,4 +19,5 @@
     <link name="base_link">
     </link>
+    <!-- FRAME LINK -->
     <joint name="frame_joint" type="fixed">
         <parent link="base_link"/>
@@ -23,8 +28,256 @@
         <visual>
             <geometry>
-                <mesh filename="file://$(find hexapod)/meshes/frame.stl" scale="0.1"/>
-                <material name="white"/>
-            </geometry>
-        </visual>
+                <mesh filename="file://$(find hexapod)/meshes/frame.stl" scale="0.001 0.001 0.001"/>
+            </geometry>
+            <material name="white"/>
+        </visual>
+        <collision>
+            <geometry>
+                <mesh filename="file://$(find hexapod)/meshes/frame.stl" scale="0.001 0.001 0.001"/>
+            </geometry>
+        </collision>
+    </link>
+    <!-- FRAME SERVOS -->
+    <joint name="servo1_joint" type="fixed">
+        <parent link="frame"/>
+        <child link="servo1"/>
+        <origin xyz="0 0 0"/>
+    </joint>
+    <link name="servo1">
+        <visual>
+            <origin xyz="0.057 0.075 0.0075" rpy="${pi/2} 0.0 ${pi/4}"/>
+            <geometry>
+                <box size="0.0405 0.0395 0.02"/>
+            </geometry>
+            <material name="black"/>
+        </visual>
+        <collision>
+            <origin xyz="0.057 0.075 0.0075" rpy="${pi/2} 0.0 ${pi/4}"/>
+            <geometry>
+                <box size="0.0405 0.0395 0.02"/>
+            </geometry>
+        </collision>
+    </link>
+    <joint name="servo2_joint" type="fixed">
+        <parent link="frame"/>
+        <child link="servo2"/>
+        <origin xyz="0 0 0"/>
+    </joint>
+    <link name="servo2">
+        <visual>
+            <origin xyz="0.07 0 0.0075" rpy="${pi/2} 0.0 0"/>
+            <geometry>
+                <box size="0.0405 0.0395 0.02"/>
+            </geometry>
+            <material name="black"/>
+        </visual>
+        <collision>
+            <origin xyz="0.07 0 0.0075" rpy="${pi/2} 0.0 0"/>
+            <geometry>
+                <box size="0.0405 0.0395 0.02"/>
+            </geometry>
+        </collision>
+    </link>
+    <joint name="servo3_joint" type="fixed">
+        <parent link="frame"/>
+        <child link="servo3"/>
+        <origin xyz="0 0 0"/>
+    </joint>
+    <link name="servo3">
+        <visual>
+            <origin xyz="0.055 -0.078 0.0075" rpy="${pi/2} 0.0 -${pi/4}"/>
+            <geometry>
+                <box size="0.0405 0.0395 0.02"/>
+            </geometry>
+            <material name="black"/>
+        </visual>
+        <collision>
+            <origin xyz="0.055 -0.078 0.0075" rpy="${pi/2} 0.0 -${pi/4}"/>
+            <geometry>
+                <box size="0.0405 0.0395 0.02"/>
+            </geometry>
+        </collision>
+    </link>
+    <joint name="servo4_joint" type="fixed">
+        <parent link="frame"/>
+        <child link="servo4"/>
+        <origin xyz="0 0 0"/>
+    </joint>
+    <link name="servo4">
+        <visual>
+            <origin xyz="-0.055 -0.078 0.0075" rpy="${pi/2} 0.0 ${pi/4}"/>
+            <geometry>
+                <box size="0.0405 0.0395 0.02"/>
+            </geometry>
+            <material name="black"/>
+        </visual>
+        <collision>
+            <origin xyz="-0.055 -0.078 0.0075" rpy="${pi/2} 0.0 ${pi/4}"/>
+            <geometry>
+                <box size="0.0405 0.0395 0.02"/>
+            </geometry>
+        </collision>
+    </link>
+    <joint name="servo5_joint" type="fixed">
+        <parent link="frame"/>
+        <child link="servo5"/>
+        <origin xyz="0 0 0"/>
+    </joint>
+    <link name="servo5">
+        <visual>
+            <origin xyz="-0.07 0 0.0075" rpy="${pi/2} 0.0 0"/>
+            <geometry>
+                <box size="0.0405 0.0395 0.02"/>
+            </geometry>
+            <material name="black"/>
+        </visual>
+        <collision>
+            <origin xyz="-0.07 0 0.0075" rpy="${pi/2} 0.0 0"/>
+            <geometry>
+                <box size="0.0405 0.0395 0.02"/>
+            </geometry>
+        </collision>
+    </link>
+    <joint name="servo6_joint" type="fixed">
+        <parent link="frame"/>
+        <child link="servo6"/>
+        <origin xyz="0 0 0"/>
+    </joint>
+    <link name="servo6">
+        <visual>
+            <origin xyz="-0.057 0.075 0.0075" rpy="${pi/2} 0.0 -${pi/4}"/>
+            <geometry>
+                <box size="0.0405 0.0395 0.02"/>
+            </geometry>
+            <material name="black"/>
+        </visual>
+        <collision>
+            <origin xyz="-0.057 0.075 0.0075" rpy="${pi/2} 0.0 -${pi/4}"/>
+            <geometry>
+                <box size="0.0405 0.0395 0.02"/>
+            </geometry>
+        </collision>
+    </link>
+    <!-- TOP -->
+    <joint name="top_cover_joint" type="fixed">
+        <parent link="frame"/>
+        <child link="top_cover"/>
+        <origin xyz="0 0 0"/>
+    </joint>
+    <link name="top_cover">
+        <visual>
+            <origin xyz="0 0 0.014"/>
+            <geometry>
+                <mesh filename="file://$(find hexapod)/meshes/top_cover.stl" scale="0.001 0.001 0.001"/>
+            </geometry>
+            <material name="blue"/>
+        </visual>
+        <collision>
+            <origin xyz="0 0 0.014"/>
+            <geometry>
+                <mesh filename="file://$(find hexapod)/meshes/top_cover.stl" scale="0.001 0.001 0.001"/>
+            </geometry>
+        </collision>
+    </link>
+    <joint name="phone_joint" type="fixed">
+        <parent link="top_cover"/>
+        <child link="phone"/>
+        <origin xyz="0 0 0"/>
+    </joint>
+    <link name="phone">
+        <visual>
+            <origin xyz="0 0 .024"/>
+            <geometry>
+                <box size="0.0699 0.1422 0.0079"/>
+            </geometry>
+            <material name="phone"/>
+        </visual>
+        <collision>
+            <origin xyz="0 0 .024"/>
+            <geometry>
+                <box size="0.0699 0.1422 0.0079"/>
+            </geometry>
+        </collision>
+    </link>
+    <!-- BOTTOM -->
+    <joint name="bottom_cover_joint" type="fixed">
+        <parent link="frame"/>
+        <child link="bottom_cover"/>
+        <origin xyz="0 0 0"/>
+    </joint>
+    <link name="bottom_cover">
+        <visual>
+            <origin xyz="0 0 .0175"/>
+            <geometry>
+                <mesh filename="file://$(find hexapod)/meshes/bottom_cover.stl" scale="0.001 0.001 0.001"/>
+            </geometry>
+            <material name="blue"/>
+        </visual>
+        <collision>
+            <origin xyz="0 0 .0175"/>
+            <geometry>
+                <mesh filename="file://$(find hexapod)/meshes/bottom_cover.stl" scale="0.001 0.001 0.001"/>
+            </geometry>
+        </collision>
+    </link>
+    <joint name="batterybar1_joint" type="fixed">
+        <parent link="bottom_cover"/>
+        <child link="batterybar1"/>
+        <origin xyz="0 0 0"/>
+    </joint>
+    <link name="batterybar1">
+        <visual>
+            <origin xyz="0 0.005 .0175"/>
+            <geometry>
+                <mesh filename="file://$(find hexapod)/meshes/battery_bar.stl" scale="0.001 0.001 0.001"/>
+            </geometry>
+            <material name="white"/>
+        </visual>
+        <collision>
+            <origin xyz="0 0.005 .0175"/>
+            <geometry>
+                <mesh filename="file://$(find hexapod)/meshes/battery_bar.stl" scale="0.001 0.001 0.001"/>
+            </geometry>
+        </collision>
+    </link>
+    <joint name="batterybar2_joint" type="fixed">
+        <parent link="bottom_cover"/>
+        <child link="batterybar2"/>
+        <origin xyz="0 0 0"/>
+    </joint>
+    <link name="batterybar2">
+        <visual>
+            <origin xyz="0 -0.075 .0175"/>
+            <geometry>
+                <mesh filename="file://$(find hexapod)/meshes/battery_bar.stl" scale="0.001 0.001 0.001"/>
+            </geometry>
+            <material name="white"/>
+        </visual>
+        <collision>
+            <origin xyz="0 -0.075 .0175"/>
+            <geometry>
+                <mesh filename="file://$(find hexapod)/meshes/battery_bar.stl" scale="0.001 0.001 0.001"/>
+            </geometry>
+        </collision>
+    </link>
+    <joint name="battery_joint" type="fixed">
+        <parent link="bottom_cover"/>
+        <child link="battery"/>
+        <origin xyz="0 0 0"/>
+    </joint>
+    <link name="battery">
+        <visual>
+            <origin xyz="0 0 -.0225"/>
+            <geometry>
+                <box size="0.047 0.138 0.025"/>
+            </geometry>
+            <material name="black"/>
+        </visual>
+        <collision>
+            <origin xyz="0 0 -.0225"/>
+            <geometry>
+                <box size="0.047 0.138 0.025"/>
+            </geometry>
+        </collision>
     </link>
 </robot>

Commit message: Update URDF with physics information

File: description/robot_frame.xacro (robot description, xacro)
@@ -1,4 +1,5 @@
 <?xml version="1.0"?>
 <robot xmlns:xacro="http://www.ros.org/wiki/xacro">
+    <xacro:include filename="inertial_macros.xacro" />
     <!-- MATERIALS -->
     <material name="white">
@@ -27,4 +28,5 @@
     <link name="frame">
         <visual>
+            <origin xyz="0 0 0"/>
             <geometry>
                 <mesh filename="file://$(find hexapod)/meshes/frame.stl" scale="0.001 0.001 0.001"/>
@@ -33,8 +35,12 @@
         </visual>
         <collision>
+            <origin xyz="0 0 0"/>
             <geometry>
                 <mesh filename="file://$(find hexapod)/meshes/frame.stl" scale="0.001 0.001 0.001"/>
             </geometry>
         </collision>
+        <xacro:inertial_box mass="0.174" x="0" y="0" z="0">
+            <origin xyz="0 0 0"/>
+        </xacro:inertial_box>
     </link>
     <!-- FRAME SERVOS -->
@@ -58,4 +64,7 @@
             </geometry>
         </collision>
+        <xacro:inertial_box mass="0.055" x="0.057" y="0.075" z="0.0075">
+            <origin xyz="0.057 0.075 0.0075" rpy="${pi/2} 0.0 ${pi/4}"/>
+        </xacro:inertial_box>
     </link>
     <joint name="servo2_joint" type="fixed">
@@ -78,4 +87,7 @@
             </geometry>
         </collision>
+        <xacro:inertial_box mass="0.055" x="0.07" y="0" z="0.0075">
+            <origin xyz="0.07 0 0.0075" rpy="${pi/2} 0.0 0"/>
+        </xacro:inertial_box>
     </link>
     <joint name="servo3_joint" type="fixed">
@@ -98,4 +110,7 @@
             </geometry>
         </collision>
+        <xacro:inertial_box mass="0.055" x="0.055" y="-0.078" z="0.0075">
+            <origin xyz="0.055 -0.078 0.0075" rpy="${pi/2} 0.0 -${pi/4}"/>
+        </xacro:inertial_box>
     </link>
     <joint name="servo4_joint" type="fixed">
@@ -118,4 +133,7 @@
             </geometry>
         </collision>
+        <xacro:inertial_box mass="0.055" x="-0.055" y="-0.078" z="0.0075">
+            <origin xyz="-0.055 -0.078 0.0075" rpy="${pi/2} 0.0 ${pi/4}"/>
+        </xacro:inertial_box>
     </link>
     <joint name="servo5_joint" type="fixed">
@@ -138,4 +156,7 @@
             </geometry>
         </collision>
+        <xacro:inertial_box mass="0.055" x="-0.07" y="0.0" z="0.0075">
+            <origin xyz="-0.07 0 0.0075" rpy="${pi/2} 0.0 0"/>
+        </xacro:inertial_box>
     </link>
     <joint name="servo6_joint" type="fixed">
@@ -158,4 +179,7 @@
             </geometry>
         </collision>
+        <xacro:inertial_box mass="0.055" x="-0.057" y="0.075" z="0.0075">
+            <origin xyz="-0.057 0.075 0.0075" rpy="${pi/2} 0.0 -${pi/4}"/>
+        </xacro:inertial_box>
     </link>
     <!-- TOP -->
@@ -179,4 +203,7 @@
             </geometry>
         </collision>
+        <xacro:inertial_box mass="0.05" x="0" y="0" z="0.014">
+            <origin xyz="0 0 0.014"/>
+        </xacro:inertial_box>
     </link>
     <joint name="phone_joint" type="fixed">
@@ -199,4 +226,7 @@
             </geometry>
         </collision>
+        <xacro:inertial_box mass="0.15" x="0" y="0" z="0.024">
+            <origin xyz="0 0 .024"/>
+        </xacro:inertial_box>
     </link>
     <!-- BOTTOM -->
@@ -220,4 +250,7 @@
             </geometry>
         </collision>
+        <xacro:inertial_box mass="0.045" x="0" y="0" z="0.0175">
+            <origin xyz="0 0 .0175"/>
+        </xacro:inertial_box>
     </link>
     <joint name="batterybar1_joint" type="fixed">
@@ -240,4 +273,7 @@
             </geometry>
         </collision>
+        <xacro:inertial_box mass="0.004" x="0" y="0" z="0.0175">
+            <origin xyz="0 0 .0175"/>
+        </xacro:inertial_box>
     </link>
     <joint name="batterybar2_joint" type="fixed">
@@ -260,4 +296,7 @@
             </geometry>
         </collision>
+        <xacro:inertial_box mass="0.004" x="0" y="-0.075" z="0.0175">
+            <origin xyz="0 -0.075 .0175"/>
+        </xacro:inertial_box>
     </link>
     <joint name="battery_joint" type="fixed">
@@ -268,5 +307,5 @@
     <link name="battery">
         <visual>
-            <origin xyz="0 0 -.0225"/>
+            <origin xyz="0 0 -0.0225"/>
             <geometry>
                 <box size="0.047 0.138 0.025"/>
@@ -275,9 +314,12 @@
         </visual>
         <collision>
-            <origin xyz="0 0 -.0225"/>
+            <origin xyz="0 0 -0.0225"/>
             <geometry>
                 <box size="0.047 0.138 0.025"/>
             </geometry>
         </collision>
+        <xacro:inertial_box mass="0.25" x="0" y="0" z="-0.0225">
+            <origin xyz="0 0 -0.0225"/>
+        </xacro:inertial_box>
     </link>
 </robot>

Commit message: URDF update checkpoint

File: description/robot_frame.xacro (robot description, xacro)
@@ -183,4 +183,125 @@
         </xacro:inertial_box>
     </link>
+    <!-- LEG SERVOS (COXA) -->
+    <joint name="coxa1_joint" type="revolute">
+        <parent link="servo1"/>
+        <child link="coxa1"/>
+        <origin xyz="0.06 0.085 -0.0025" rpy="0 0 ${pi/4}"/>
+        <axis xyz="0 0 1" />
+        <limit lower="-0.785398" upper="0.785398" effort="0.8825985000000001" velocity="1.0"/>
+    </joint>
+    <link name="coxa1">
+        <visual>
+            <origin xyz="0 0 -0.0025"/>
+            <geometry>
+                <mesh filename="file://$(find hexapod)/meshes/right_coxa.stl" scale="0.001 0.001 0.001"/>
+            </geometry>
+            <material name="white"/>
+        </visual>
+    </link>
+    <joint name="servo7_joint" type="fixed">
+        <parent link="coxa1"/>
+        <child link="servo7"/>
+        <origin xyz="0 0 0"/>
+    </joint>
+    <link name="servo7">
+        <visual>
+            <origin xyz="0.045 0 0.0095" rpy="0 ${pi/2} 0"/>
+            <geometry>
+                <box size="0.0405 0.0395 0.02"/>
+            </geometry>
+            <material name="black"/>
+        </visual>
+        <collision>
+            <origin xyz="0.045 0 0.0095" rpy="0 ${pi/2} 0"/>
+            <geometry>
+                <box size="0.0405 0.0395 0.02"/>
+            </geometry>
+        </collision>
+        <xacro:inertial_box mass="0.055" x="0.045" y="0" z="0.0095">
+            <origin xyz="0.045 0 0.0095" rpy="0 ${pi/2} 0"/>
+        </xacro:inertial_box>
+    </link>
+    <joint name="coxa2_joint" type="revolute">
+        <parent link="servo2"/>
+        <child link="coxa2"/>
+        <origin xyz="0.08 0 -0.0025"/>
+        <axis xyz="0 0 1" />
+        <limit lower="-0.785398" upper="0.785398" effort="0.8825985000000001" velocity="1.0"/>
+    </joint>
+    <link name="coxa2">
+        <visual>
+            <origin xyz="0 0 -0.0025"/>
+            <geometry>
+                <mesh filename="file://$(find hexapod)/meshes/right_coxa.stl" scale="0.001 0.001 0.001"/>
+            </geometry>
+            <material name="white"/>
+        </visual>
+    </link>
+    <joint name="coxa3_joint" type="revolute">
+        <parent link="servo3"/>
+        <child link="coxa3"/>
+        <origin xyz="0.06 -0.085 -0.0025" rpy="0 0 -${pi/4}"/>
+        <axis xyz="0 0 1" />
+        <limit lower="-0.785398" upper="0.785398" effort="0.8825985000000001" velocity="1.0"/>
+    </joint>
+    <link name="coxa3">
+        <visual>
+            <origin xyz="0 0 -0.0025"/>
+            <geometry>
+                <mesh filename="file://$(find hexapod)/meshes/right_coxa.stl" scale="0.001 0.001 0.001"/>
+            </geometry>
+            <material name="white"/>
+        </visual>
+    </link>
+    <joint name="coxa4_joint" type="revolute">
+        <parent link="servo4"/>
+        <child link="coxa4"/>
+        <origin xyz="-0.06 -0.085 -0.0025" rpy="0 0 -${(3*pi)/4}"/>
+        <axis xyz="0 0 1" />
+        <limit lower="-0.785398" upper="0.785398" effort="0.8825985000000001" velocity="1.0"/>
+    </joint>
+    <link name="coxa4">
+        <visual>
+            <origin xyz="0 0 -0.0025"/>
+            <geometry>
+                <mesh filename="file://$(find hexapod)/meshes/right_coxa.stl" scale="0.001 0.001 0.001"/>
+            </geometry>
+            <material name="white"/>
+        </visual>
+    </link>
+    <joint name="coxa5_joint" type="revolute">
+        <parent link="servo5"/>
+        <child link="coxa5"/>
+        <origin xyz="-0.08 0 -0.0025" rpy="0 0 ${pi}"/>
+        <axis xyz="0 0 1" />
+        <limit lower="-0.785398" upper="0.785398" effort="0.8825985000000001" velocity="1.0"/>
+    </joint>
+    <link name="coxa5">
+        <visual>
+            <origin xyz="0 0 -0.0025"/>
+            <geometry>
+                <mesh filename="file://$(find hexapod)/meshes/left_coxa.stl" scale="0.001 0.001 0.001"/>
+            </geometry>
+            <material name="white"/>
+        </visual>
+    </link>
+    <joint name="coxa6_joint" type="revolute">
+        <parent link="servo6"/>
+        <child link="coxa6"/>
+        <origin xyz="-0.06 0.085 0" rpy="0 0 ${(3*pi)/4}"/>
+        <axis xyz="0 0 1" />
+        <limit lower="-0.785398" upper="0.785398" effort="0.8825985000000001" velocity="1.0"/>
+    </joint>
+    <link name="coxa6">
+        <visual>
+            <origin xyz="0 0 -0.005"/>
+            <geometry>
+                <mesh filename="file://$(find hexapod)/meshes/left_coxa.stl" scale="0.001 0.001 0.001"/>
+            </geometry>
+            <material name="white"/>
+        </visual>
+    </link>
+    <!-- LEG SERVOS (FEMUR) -->
     <!-- TOP -->
     <joint name="top_cover_joint" type="fixed">
