Commit message: URDF Tibia addition checkpoint

File: description/robot_frame.xacro (robot description, xacro)
@@ -64,5 +64,5 @@
             </geometry>
         </collision>
-        <xacro:inertial_box mass="0.055" x="0.057" y="0.075" z="0.0075">
+        <xacro:inertial_box mass="0.055" x="0.0405" y="0.0395" z="0.02">
             <origin xyz="0.057 0.075 0.0075" rpy="${pi/2} 0.0 ${pi/4}"/>
         </xacro:inertial_box>
@@ -87,5 +87,5 @@
             </geometry>
         </collision>
-        <xacro:inertial_box mass="0.055" x="0.07" y="0" z="0.0075">
+        <xacro:inertial_box mass="0.055" x="0.0405" y="0.0395" z="0.02">
             <origin xyz="0.07 0 0.0075" rpy="${pi/2} 0.0 0"/>
         </xacro:inertial_box>
@@ -110,5 +110,5 @@
             </geometry>
         </collision>
-        <xacro:inertial_box mass="0.055" x="0.055" y="-0.078" z="0.0075">
+        <xacro:inertial_box mass="0.055" x="0.0405" y="0.0395" z="0.02">
             <origin xyz="0.055 -0.078 0.0075" rpy="${pi/2} 0.0 -${pi/4}"/>
         </xacro:inertial_box>
@@ -133,5 +133,5 @@
             </geometry>
         </collision>
-        <xacro:inertial_box mass="0.055" x="-0.055" y="-0.078" z="0.0075">
+        <xacro:inertial_box mass="0.055" x="0.0405" y="0.0395" z="0.02">
             <origin xyz="-0.055 -0.078 0.0075" rpy="${pi/2} 0.0 ${pi/4}"/>
         </xacro:inertial_box>
@@ -156,5 +156,5 @@
             </geometry>
         </collision>
-        <xacro:inertial_box mass="0.055" x="-0.07" y="0.0" z="0.0075">
+        <xacro:inertial_box mass="0.055" x="0.0405" y="0.0395" z="0.02">
             <origin xyz="-0.07 0 0.0075" rpy="${pi/2} 0.0 0"/>
         </xacro:inertial_box>
@@ -179,6 +179,6 @@
             </geometry>
         </collision>
-        <xacro:inertial_box mass="0.055" x="-0.057" y="0.075" z="0.0075">
-            <origin xyz="-0.057 0.075 0.0075" rpy="${pi/2} 0.0 -${pi/4}"/>
+        <xacro:inertial_box mass="0.055" x="0.0405" y="0.0395" z="0.02">
+            <origin xyz="-0.057 0.075 0.0075"/>
         </xacro:inertial_box>
     </link>
@@ -200,4 +200,13 @@
             <material name="white"/>
         </visual>
+        <collision>
+            <origin xyz="0 0 -0.0025"/>
+            <geometry>
+                <mesh filename="file://$(find hexapod)/meshes/right_coxa.stl" scale="0.001 0.001 0.001"/>
+            </geometry>
+        </collision>
+        <xacro:inertial_box mass="0.015" x="0.01" y="0.01" z="0.01">
+            <origin xyz="0.025 0 0.0025" rpy="0 0 0"/>
+        </xacro:inertial_box>
     </link>
     <joint name="servo7_joint" type="fixed">
@@ -220,5 +229,5 @@
             </geometry>
         </collision>
-        <xacro:inertial_box mass="0.055" x="0.045" y="0" z="0.0095">
+        <xacro:inertial_box mass="0.055" x="0.0405" y="0.0395" z="0.02">
             <origin xyz="0.045 0 0.0095" rpy="0 ${pi/2} 0"/>
         </xacro:inertial_box>
@@ -236,4 +245,52 @@
             <geometry>
                 <mesh filename="file://$(find hexapod)/meshes/right_femur.stl" scale="0.001 0.001 0.001"/>
+            </geometry>
+            <material name="white"/>
+        </visual>
+        <collision>
+             <origin xyz="-0.08 0 -0.0125"/>
+            <geometry>
+                <mesh filename="file://$(find hexapod)/meshes/right_femur.stl" scale="0.001 0.001 0.001"/>
+            </geometry>
+        </collision>
+        <xacro:inertial_box mass="0.015" x="0.01" y="0.01" z="0.01">
+             <origin xyz="-0.08 0 -0.0125"/>
+        </xacro:inertial_box>
+    </link>
+    <joint name="servo13_joint" type="revolute">
+        <parent link="femur1"/>
+        <child link="servo13"/>
+        <origin xyz="-0.0775 0 0"/>
+        <axis xyz="0 0 1" />
+        <limit lower="-0.785398" upper="0.785398" effort="0.8825985000000001" velocity="1.0"/>
+    </joint>
+    <link name="servo13">
+        <visual>
+            <origin xyz="-0.008 0 0" rpy="${pi/2} ${pi/2} 0"/>
+            <geometry>
+                <box size="0.0405 0.0395 0.02"/>
+            </geometry>
+            <material name="black"/>
+        </visual>
+        <collision>
+            <origin xyz="-0.008 0 0" rpy="${pi/2} ${pi/2} 0"/>
+            <geometry>
+                <box size="0.0405 0.0395 0.02"/>
+            </geometry>
+        </collision>
+        <xacro:inertial_box mass="0.055" x="0.0405" y="0.0395" z="0.02">
+            <origin xyz="-0.008 0 0" rpy="${pi/2} ${pi/2} 0"/>
+        </xacro:inertial_box>
+    </link>
+    <joint name="tibia1_joint" type="fixed">
+        <parent link="servo13"/>
+        <child link="tibia1"/>
+        <origin xyz="0 0 0" rpy="-${pi/2} 0 -0.85"/>
+    </joint>
+    <link name="tibia1">
+        <visual>
+            <origin xyz="-0.055 0 0.005"/>
+            <geometry>
+                <mesh filename="file://$(find hexapod)/meshes/right_tibia.stl" scale="0.001 0.001 0.001"/>
             </geometry>
             <material name="white"/>
@@ -256,4 +313,13 @@
             <material name="white"/>
         </visual>
+        <collision>
+            <origin xyz="0 0 -0.0025"/>
+            <geometry>
+                <mesh filename="file://$(find hexapod)/meshes/right_coxa.stl" scale="0.001 0.001 0.001"/>
+            </geometry>
+        </collision>
+        <xacro:inertial_box mass="0.015" x="0.01" y="0.01" z="0.01">
+            <origin xyz="0.025 0 0.0025" rpy="0 0 0"/>
+        </xacro:inertial_box>
     </link>
     <joint name="servo8_joint" type="fixed">
@@ -276,5 +342,5 @@
             </geometry>
         </collision>
-        <xacro:inertial_box mass="0.055" x="0.045" y="0" z="0.0095">
+        <xacro:inertial_box mass="0.055" x="0.0405" y="0.0395" z="0.02">
             <origin xyz="0.045 0 0.0095" rpy="0 ${pi/2} 0"/>
         </xacro:inertial_box>
@@ -292,4 +358,52 @@
             <geometry>
                 <mesh filename="file://$(find hexapod)/meshes/right_femur.stl" scale="0.001 0.001 0.001"/>
+            </geometry>
+            <material name="white"/>
+        </visual>
+        <collision>
+             <origin xyz="-0.08 0 -0.0125"/>
+            <geometry>
+                <mesh filename="file://$(find hexapod)/meshes/right_femur.stl" scale="0.001 0.001 0.001"/>
+            </geometry>
+        </collision>
+        <xacro:inertial_box mass="0.015" x="0.01" y="0.01" z="0.01">
+             <origin xyz="-0.08 0 -0.0125"/>
+        </xacro:inertial_box>
+    </link>
+    <joint name="servo14_joint" type="revolute">
+        <parent link="femur2"/>
+        <child link="servo14"/>
+        <origin xyz="-0.0775 0 0"/>
+        <axis xyz="0 0 1" />
+        <limit lower="-0.785398" upper="0.785398" effort="0.8825985000000001" velocity="1.0"/>
+    </joint>
+    <link name="servo14">
+        <visual>
+            <origin xyz="-0.008 0 0" rpy="${pi/2} ${pi/2} 0"/>
+            <geometry>
+                <box size="0.0405 0.0395 0.02"/>
+            </geometry>
+            <material name="black"/>
+        </visual>
+        <collision>
+            <origin xyz="-0.008 0 0" rpy="${pi/2} ${pi/2} 0"/>
+            <geometry>
+                <box size="0.0405 0.0395 0.02"/>
+            </geometry>
+        </collision>
+        <xacro:inertial_box mass="0.055" x="0.0405" y="0.0395" z="0.02">
+            <origin xyz="-0.008 0 0" rpy="${pi/2} ${pi/2} 0"/>
+        </xacro:inertial_box>
+    </link>
+    <joint name="tibia2_joint" type="fixed">
+        <parent link="servo14"/>
+        <child link="tibia2"/>
+        <origin xyz="0 0 0" rpy="-${pi/2} 0 -0.85"/>
+    </joint>
+    <link name="tibia2">
+        <visual>
+            <origin xyz="-0.055 0 0.005"/>
+            <geometry>
+                <mesh filename="file://$(find hexapod)/meshes/right_tibia.stl" scale="0.001 0.001 0.001"/>
             </geometry>
             <material name="white"/>
@@ -312,4 +426,13 @@
             <material name="white"/>
         </visual>
+        <collision>
+            <origin xyz="0 0 -0.0025"/>
+            <geometry>
+                <mesh filename="file://$(find hexapod)/meshes/right_coxa.stl" scale="0.001 0.001 0.001"/>
+            </geometry>
+        </collision>
+        <xacro:inertial_box mass="0.015" x="0.01" y="0.01" z="0.01">
+            <origin xyz="0 0 0.0025" rpy="0 0 0"/>
+        </xacro:inertial_box>
     </link>
     <joint name="servo9_joint" type="fixed">
@@ -332,5 +455,5 @@
             </geometry>
         </collision>
-        <xacro:inertial_box mass="0.055" x="0.045" y="0" z="0.0095">
+        <xacro:inertial_box mass="0.055" x="0.0405" y="0.0395" z="0.02">
             <origin xyz="0.045 0 0.0095" rpy="0 ${pi/2} 0"/>
         </xacro:inertial_box>
@@ -348,4 +471,52 @@
             <geometry>
                 <mesh filename="file://$(find hexapod)/meshes/right_femur.stl" scale="0.001 0.001 0.001"/>
+            </geometry>
+            <material name="white"/>
+        </visual>
+        <collision>
+             <origin xyz="-0.08 0 -0.0125"/>
+            <geometry>
+                <mesh filename="file://$(find hexapod)/meshes/right_femur.stl" scale="0.001 0.001 0.001"/>
+            </geometry>
+        </collision>
+        <xacro:inertial_box mass="0.015" x="0.01" y="0.01" z="0.01">
+             <origin xyz="-0.08 0 -0.0125"/>
+        </xacro:inertial_box>
+    </link>
+    <joint name="servo15_joint" type="revolute">
+        <parent link="femur3"/>
+        <child link="servo15"/>
+        <origin xyz="-0.0775 0 0"/>
+        <axis xyz="0 0 1" />
+        <limit lower="-0.785398" upper="0.785398" effort="0.8825985000000001" velocity="1.0"/>
+    </joint>
+    <link name="servo15">
+        <visual>
+            <origin xyz="-0.008 0 0" rpy="${pi/2} ${pi/2} 0"/>
+            <geometry>
+                <box size="0.0405 0.0395 0.02"/>
+            </geometry>
+            <material name="black"/>
+        </visual>
+        <collision>
+            <origin xyz="-0.008 0 0" rpy="${pi/2} ${pi/2} 0"/>
+            <geometry>
+                <box size="0.0405 0.0395 0.02"/>
+            </geometry>
+        </collision>
+        <xacro:inertial_box mass="0.055" x="0.0405" y="0.0395" z="0.02">
+            <origin xyz="-0.008 0 0" rpy="${pi/2} ${pi/2} 0"/>
+        </xacro:inertial_box>
+    </link>
+    <joint name="tibia3_joint" type="fixed">
+        <parent link="servo15"/>
+        <child link="tibia3"/>
+        <origin xyz="0 0 0" rpy="-${pi/2} 0 -0.85"/>
+    </joint>
+    <link name="tibia3">
+        <visual>
+            <origin xyz="-0.055 0 0.005"/>
+            <geometry>
+                <mesh filename="file://$(find hexapod)/meshes/right_tibia.stl" scale="0.001 0.001 0.001"/>
             </geometry>
             <material name="white"/>
@@ -364,8 +535,17 @@
             <origin xyz="0 0 -0.0025"/>
             <geometry>
-                <mesh filename="file://$(find hexapod)/meshes/right_coxa.stl" scale="0.001 0.001 0.001"/>
-            </geometry>
-            <material name="white"/>
-        </visual>
+                <mesh filename="file://$(find hexapod)/meshes/left_coxa.stl" scale="0.001 0.001 0.001"/>
+            </geometry>
+            <material name="white"/>
+        </visual>
+        <collision>
+            <origin xyz="0 0 -0.0025"/>
+            <geometry>
+                <mesh filename="file://$(find hexapod)/meshes/left_coxa.stl" scale="0.001 0.001 0.001"/>
+            </geometry>
+        </collision>
+        <xacro:inertial_box mass="0.015" x="0.01" y="0.01" z="0.01">
+            <origin xyz="0 0 0.0025" rpy="0 0 0"/>
+        </xacro:inertial_box>
     </link>
     <joint name="servo10_joint" type="fixed">
@@ -388,5 +568,5 @@
             </geometry>
         </collision>
-        <xacro:inertial_box mass="0.055" x="0.045" y="0" z="0.0095">
+        <xacro:inertial_box mass="0.055" x="0.0405" y="0.0395" z="0.02">
             <origin xyz="0.045 0 0.0095" rpy="0 ${pi/2} 0"/>
         </xacro:inertial_box>
@@ -404,4 +584,52 @@
             <geometry>
                 <mesh filename="file://$(find hexapod)/meshes/left_femur.stl" scale="0.001 0.001 0.001"/>
+            </geometry>
+            <material name="white"/>
+        </visual>
+        <collision>
+             <origin xyz="-0.08 0 -0.0125"/>
+            <geometry>
+                <mesh filename="file://$(find hexapod)/meshes/left_femur.stl" scale="0.001 0.001 0.001"/>
+            </geometry>
+        </collision>
+        <xacro:inertial_box mass="0.015" x="0.01" y="0.01" z="0.01">
+             <origin xyz="-0.08 0 -0.0125"/>
+        </xacro:inertial_box>
+    </link>
+    <joint name="servo16_joint" type="revolute">
+        <parent link="femur4"/>
+        <child link="servo16"/>
+        <origin xyz="-0.0775 0 0"/>
+        <axis xyz="0 0 1" />
+        <limit lower="-0.785398" upper="0.785398" effort="0.8825985000000001" velocity="1.0"/>
+    </joint>
+    <link name="servo16">
+        <visual>
+            <origin xyz="-0.008 0 0" rpy="${pi/2} ${pi/2} 0"/>
+            <geometry>
+                <box size="0.0405 0.0395 0.02"/>
+            </geometry>
+            <material name="black"/>
+        </visual>
+        <collision>
+            <origin xyz="-0.008 0 0" rpy="${pi/2} ${pi/2} 0"/>
+            <geometry>
+                <box size="0.0405 0.0395 0.02"/>
+            </geometry>
+        </collision>
+        <xacro:inertial_box mass="0.055" x="0.0405" y="0.0395" z="0.02">
+            <origin xyz="-0.008 0 0" rpy="${pi/2} ${pi/2} 0"/>
+        </xacro:inertial_box>
+    </link>
+    <joint name="tibia4_joint" type="fixed">
+        <parent link="servo16"/>
+        <child link="tibia4"/>
+        <origin xyz="0 0 0" rpy="-${pi/2} 0 -0.85"/>
+    </joint>
+    <link name="tibia4">
+        <visual>
+            <origin xyz="-0.055 0 0.005"/>
+            <geometry>
+                <mesh filename="file://$(find hexapod)/meshes/left_tibia.stl" scale="0.001 0.001 0.001"/>
             </geometry>
             <material name="white"/>
@@ -424,4 +652,13 @@
             <material name="white"/>
         </visual>
+        <collision>
+            <origin xyz="0 0 -0.0025"/>
+            <geometry>
+                <mesh filename="file://$(find hexapod)/meshes/left_coxa.stl" scale="0.001 0.001 0.001"/>
+            </geometry>
+        </collision>
+        <xacro:inertial_box mass="0.015" x="0.01" y="0.01" z="0.01">
+            <origin xyz="0 0 0.0025" rpy="0 0 0"/>
+        </xacro:inertial_box>
     </link>
     <joint name="servo11_joint" type="fixed">
@@ -444,5 +681,5 @@
             </geometry>
         </collision>
-        <xacro:inertial_box mass="0.055" x="0.045" y="0" z="0.0095">
+        <xacro:inertial_box mass="0.055" x="0.0405" y="0.0395" z="0.02">
             <origin xyz="0.045 0 0.0095" rpy="0 ${pi/2} 0"/>
         </xacro:inertial_box>
@@ -460,4 +697,52 @@
             <geometry>
                 <mesh filename="file://$(find hexapod)/meshes/left_femur.stl" scale="0.001 0.001 0.001"/>
+            </geometry>
+            <material name="white"/>
+        </visual>
+        <collision>
+             <origin xyz="-0.08 0 -0.0125"/>
+            <geometry>
+                <mesh filename="file://$(find hexapod)/meshes/left_femur.stl" scale="0.001 0.001 0.001"/>
+            </geometry>
+        </collision>
+        <xacro:inertial_box mass="0.015" x="0.01" y="0.01" z="0.01">
+             <origin xyz="-0.08 0 -0.0125"/>
+        </xacro:inertial_box>
+    </link>
+    <joint name="servo17_joint" type="revolute">
+        <parent link="femur5"/>
+        <child link="servo17"/>
+        <origin xyz="-0.0775 0 0"/>
+        <axis xyz="0 0 1" />
+        <limit lower="-0.785398" upper="0.785398" effort="0.8825985000000001" velocity="1.0"/>
+    </joint>
+    <link name="servo17">
+        <visual>
+            <origin xyz="-0.008 0 0" rpy="${pi/2} ${pi/2} 0"/>
+            <geometry>
+                <box size="0.0405 0.0395 0.02"/>
+            </geometry>
+            <material name="black"/>
+        </visual>
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