Commit message: URDF model update

File: description/robot_frame.xacro (robot description, xacro)
@@ -236,5 +236,5 @@
         <parent link="servo7"/>
         <child link="femur1"/>
-        <origin xyz="0.045 0 0.02" rpy="${pi/2} 0 ${pi}"/>
+        <origin xyz="0.045 0 0.02" rpy="${pi/2} ${pi/4} ${pi}"/>
         <axis xyz="0 0 1" />
         <limit lower="-0.785398" upper="0.785398" effort="0.8825985000000001" velocity="1.0"/>
@@ -261,5 +261,5 @@
         <parent link="femur1"/>
         <child link="servo13"/>
-        <origin xyz="-0.0775 0 0"/>
+        <origin xyz="-0.0775 0 0" rpy="0 0 ${pi/4}"/>
         <axis xyz="0 0 1" />
         <limit lower="-0.785398" upper="0.785398" effort="0.8825985000000001" velocity="1.0"/>
@@ -296,4 +296,59 @@
             <material name="white"/>
         </visual>
+        <collision>
+            <origin xyz="-0.055 0 0.005"/>
+            <geometry>
+                <mesh filename="file://$(find hexapod)/meshes/right_tibia.stl" scale="0.001 0.001 0.001"/>
+            </geometry>
+        </collision>
+        <xacro:inertial_box mass="0.015" x="0.01" y="0.01" z="0.01">
+             <origin xyz="-0.055 0 0.005"/>
+        </xacro:inertial_box>
+    </link>
+    <joint name="shield1_joint" type="fixed">
+        <parent link="tibia1"/>
+        <child link="shield1"/>
+        <origin xyz="0 0 0" rpy="0 0 0"/>
+    </joint>
+    <link name="shield1">
+        <visual>
+            <origin xyz="-0.055 0 0"/>
+            <geometry>
+                <mesh filename="file://$(find hexapod)/meshes/shield.stl" scale="0.001 0.001 0.001"/>
+            </geometry>
+            <material name="blue"/>
+        </visual>
+        <collision>
+            <origin xyz="-0.055 0 0"/>
+            <geometry>
+                <mesh filename="file://$(find hexapod)/meshes/shield.stl" scale="0.001 0.001 0.001"/>
+            </geometry>
+        </collision>
+        <xacro:inertial_box mass="0.015" x="0.01" y="0.01" z="0.01">
+             <origin xyz="-0.055 0 0"/>
+        </xacro:inertial_box>
+    </link>
+    <joint name="sensor1_joint" type="fixed">
+        <parent link="tibia1"/>
+        <child link="sensor1"/>
+        <origin xyz="0 0 0" rpy="0 0 0"/>
+    </joint>
+    <link name="sensor1">
+        <visual>
+            <origin xyz="-0.0425 0.005 -0.125"/>
+            <geometry>
+                <mesh filename="file://$(find hexapod)/meshes/micro_switch_tip.stl" scale="0.001 0.001 0.001"/>
+            </geometry>
+            <material name="white"/>
+        </visual>
+        <collision>
+            <origin xyz="-0.0425 0.005 -0.125"/>
+            <geometry>
+                <mesh filename="file://$(find hexapod)/meshes/micro_switch_tip.stl" scale="0.001 0.001 0.001"/>
+            </geometry>
+        </collision>
+        <xacro:inertial_box mass="0.015" x="0.01" y="0.01" z="0.01">
+             <origin xyz="-0.0425 0.005 -0.125"/>
+        </xacro:inertial_box>
     </link>
     <!-- LEG 2 (RM) -->
@@ -349,5 +404,5 @@
         <parent link="servo8"/>
         <child link="femur2"/>
-        <origin xyz="0.045 0 0.02" rpy="${pi/2} 0 ${pi}"/>
+        <origin xyz="0.045 0 0.02" rpy="${pi/2} ${pi/4} ${pi}"/>
         <axis xyz="0 0 1" />
         <limit lower="-0.785398" upper="0.785398" effort="0.8825985000000001" velocity="1.0"/>
@@ -374,5 +429,5 @@
         <parent link="femur2"/>
         <child link="servo14"/>
-        <origin xyz="-0.0775 0 0"/>
+        <origin xyz="-0.0775 0 0" rpy="0 0 ${pi/4}"/>
         <axis xyz="0 0 1" />
         <limit lower="-0.785398" upper="0.785398" effort="0.8825985000000001" velocity="1.0"/>
@@ -409,4 +464,59 @@
             <material name="white"/>
         </visual>
+        <collision>
+            <origin xyz="-0.055 0 0.005"/>
+            <geometry>
+                <mesh filename="file://$(find hexapod)/meshes/right_tibia.stl" scale="0.001 0.001 0.001"/>
+            </geometry>
+        </collision>
+        <xacro:inertial_box mass="0.015" x="0.01" y="0.01" z="0.01">
+             <origin xyz="-0.055 0 0.005"/>
+        </xacro:inertial_box>
+    </link>
+    <joint name="shield2_joint" type="fixed">
+        <parent link="tibia2"/>
+        <child link="shield2"/>
+        <origin xyz="0 0 0" rpy="0 0 0"/>
+    </joint>
+    <link name="shield2">
+        <visual>
+            <origin xyz="-0.055 0 0"/>
+            <geometry>
+                <mesh filename="file://$(find hexapod)/meshes/shield.stl" scale="0.001 0.001 0.001"/>
+            </geometry>
+            <material name="blue"/>
+        </visual>
+        <collision>
+            <origin xyz="-0.055 0 0"/>
+            <geometry>
+                <mesh filename="file://$(find hexapod)/meshes/shield.stl" scale="0.001 0.001 0.001"/>
+            </geometry>
+        </collision>
+        <xacro:inertial_box mass="0.015" x="0.01" y="0.01" z="0.01">
+            <origin xyz="-0.055 0 0"/>
+        </xacro:inertial_box>
+    </link>
+    <joint name="sensor2_joint" type="fixed">
+        <parent link="tibia2"/>
+        <child link="sensor2"/>
+        <origin xyz="0 0 0" rpy="0 0 0"/>
+    </joint>
+    <link name="sensor2">
+        <visual>
+            <origin xyz="-0.0425 0.005 -0.125"/>
+            <geometry>
+                <mesh filename="file://$(find hexapod)/meshes/micro_switch_tip.stl" scale="0.001 0.001 0.001"/>
+            </geometry>
+            <material name="white"/>
+        </visual>
+        <collision>
+            <origin xyz="-0.0425 0.005 -0.125"/>
+            <geometry>
+                <mesh filename="file://$(find hexapod)/meshes/micro_switch_tip.stl" scale="0.001 0.001 0.001"/>
+            </geometry>
+        </collision>
+        <xacro:inertial_box mass="0.015" x="0.01" y="0.01" z="0.01">
+             <origin xyz="-0.0425 0.005 -0.125"/>
+        </xacro:inertial_box>
     </link>
     <!-- LEG 3 (RB) -->
@@ -462,5 +572,5 @@
         <parent link="servo9"/>
         <child link="femur3"/>
-        <origin xyz="0.045 0 0.02" rpy="${pi/2} 0 ${pi}"/>
+        <origin xyz="0.045 0 0.02" rpy="${pi/2} ${pi/4} ${pi}"/>
         <axis xyz="0 0 1" />
         <limit lower="-0.785398" upper="0.785398" effort="0.8825985000000001" velocity="1.0"/>
@@ -487,5 +597,5 @@
         <parent link="femur3"/>
         <child link="servo15"/>
-        <origin xyz="-0.0775 0 0"/>
+        <origin xyz="-0.0775 0 0" rpy="0 0 ${pi/4}"/>
         <axis xyz="0 0 1" />
         <limit lower="-0.785398" upper="0.785398" effort="0.8825985000000001" velocity="1.0"/>
@@ -522,4 +632,59 @@
             <material name="white"/>
         </visual>
+        <collision>
+            <origin xyz="-0.055 0 0.005"/>
+            <geometry>
+                <mesh filename="file://$(find hexapod)/meshes/right_tibia.stl" scale="0.001 0.001 0.001"/>
+            </geometry>
+        </collision>
+        <xacro:inertial_box mass="0.015" x="0.01" y="0.01" z="0.01">
+            <origin xyz="-0.055 0 0.005"/>
+        </xacro:inertial_box>
+    </link>
+    <joint name="shield3_joint" type="fixed">
+        <parent link="tibia3"/>
+        <child link="shield3"/>
+        <origin xyz="0 0 0" rpy="0 0 0"/>
+    </joint>
+    <link name="shield3">
+        <visual>
+            <origin xyz="-0.055 0 0"/>
+            <geometry>
+                <mesh filename="file://$(find hexapod)/meshes/shield.stl" scale="0.001 0.001 0.001"/>
+            </geometry>
+            <material name="blue"/>
+        </visual>
+        <collision>
+            <origin xyz="-0.055 0 0"/>
+            <geometry>
+                <mesh filename="file://$(find hexapod)/meshes/shield.stl" scale="0.001 0.001 0.001"/>
+            </geometry>
+        </collision>
+        <xacro:inertial_box mass="0.015" x="0.01" y="0.01" z="0.01">
+            <origin xyz="-0.055 0 0"/>
+        </xacro:inertial_box>
+    </link>
+    <joint name="sensor3_joint" type="fixed">
+        <parent link="tibia3"/>
+        <child link="sensor3"/>
+        <origin xyz="0 0 0" rpy="0 0 0"/>
+    </joint>
+    <link name="sensor3">
+        <visual>
+            <origin xyz="-0.0425 0.005 -0.125"/>
+            <geometry>
+                <mesh filename="file://$(find hexapod)/meshes/micro_switch_tip.stl" scale="0.001 0.001 0.001"/>
+            </geometry>
+            <material name="white"/>
+        </visual>
+        <collision>
+            <origin xyz="-0.0425 0.005 -0.125"/>
+            <geometry>
+                <mesh filename="file://$(find hexapod)/meshes/micro_switch_tip.stl" scale="0.001 0.001 0.001"/>
+            </geometry>
+        </collision>
+        <xacro:inertial_box mass="0.015" x="0.01" y="0.01" z="0.01">
+             <origin xyz="-0.0425 0.005 -0.125"/>
+        </xacro:inertial_box>
     </link>
     <!-- LEG 4 (LB) -->
@@ -575,5 +740,5 @@
         <parent link="servo10"/>
         <child link="femur4"/>
-        <origin xyz="0.045 0 0.02" rpy="${pi/2} 0 ${pi}"/>
+        <origin xyz="0.045 0 0.02" rpy="${pi/2} ${pi/4} ${pi}"/>
         <axis xyz="0 0 1" />
         <limit lower="-0.785398" upper="0.785398" effort="0.8825985000000001" velocity="1.0"/>
@@ -600,5 +765,5 @@
         <parent link="femur4"/>
         <child link="servo16"/>
-        <origin xyz="-0.0775 0 0"/>
+        <origin xyz="-0.0775 0 0" rpy="0 0 ${pi/4}"/>
         <axis xyz="0 0 1" />
         <limit lower="-0.785398" upper="0.785398" effort="0.8825985000000001" velocity="1.0"/>
@@ -635,4 +800,59 @@
             <material name="white"/>
         </visual>
+        <collision>
+            <origin xyz="-0.055 0 0.005"/>
+            <geometry>
+                <mesh filename="file://$(find hexapod)/meshes/left_tibia.stl" scale="0.001 0.001 0.001"/>
+            </geometry>
+        </collision>
+        <xacro:inertial_box mass="0.015" x="0.01" y="0.01" z="0.01">
+            <origin xyz="-0.055 0 0.005"/>
+        </xacro:inertial_box>
+    </link>
+    <joint name="shield4_joint" type="fixed">
+        <parent link="tibia4"/>
+        <child link="shield4"/>
+        <origin xyz="0 0 0" rpy="0 0 0"/>
+    </joint>
+    <link name="shield4">
+        <visual>
+            <origin xyz="-0.055 -0.01 0"/>
+            <geometry>
+                <mesh filename="file://$(find hexapod)/meshes/shield.stl" scale="0.001 0.001 0.001"/>
+            </geometry>
+            <material name="blue"/>
+        </visual>
+        <collision>
+            <origin xyz="-0.055 -0.01 0"/>
+            <geometry>
+                <mesh filename="file://$(find hexapod)/meshes/shield.stl" scale="0.001 0.001 0.001"/>
+            </geometry>
+        </collision>
+        <xacro:inertial_box mass="0.015" x="0.01" y="0.01" z="0.01">
+            <origin xyz="-0.055 -0.01 0"/>
+        </xacro:inertial_box>
+    </link>
+    <joint name="sensor4_joint" type="fixed">
+        <parent link="tibia4"/>
+        <child link="sensor4"/>
+        <origin xyz="0 0 0" rpy="0 0 0"/>
+    </joint>
+    <link name="sensor4">
+        <visual>
+            <origin xyz="-0.0425 -0.005 -0.125"/>
+            <geometry>
+                <mesh filename="file://$(find hexapod)/meshes/micro_switch_tip.stl" scale="0.001 0.001 0.001"/>
+            </geometry>
+            <material name="white"/>
+        </visual>
+        <collision>
+            <origin xyz="-0.0425 -0.005 -0.125"/>
+            <geometry>
+                <mesh filename="file://$(find hexapod)/meshes/micro_switch_tip.stl" scale="0.001 0.001 0.001"/>
+            </geometry>
+        </collision>
+        <xacro:inertial_box mass="0.015" x="0.01" y="0.01" z="0.01">
+             <origin xyz="-0.0425 -0.005 -0.125"/>
+        </xacro:inertial_box>
     </link>
     <!-- LEG 5 (LM) -->
@@ -688,5 +908,5 @@
         <parent link="servo11"/>
         <child link="femur5"/>
-        <origin xyz="0.045 0 0.02" rpy="${pi/2} 0 ${pi}"/>
+        <origin xyz="0.045 0 0.02" rpy="${pi/2} ${pi/4} ${pi}"/>
         <axis xyz="0 0 1" />
         <limit lower="-0.785398" upper="0.785398" effort="0.8825985000000001" velocity="1.0"/>
@@ -713,5 +933,5 @@
         <parent link="femur5"/>
         <child link="servo17"/>
-        <origin xyz="-0.0775 0 0"/>
+        <origin xyz="-0.0775 0 0" rpy="0 0 ${pi/4}"/>
         <axis xyz="0 0 1" />
         <limit lower="-0.785398" upper="0.785398" effort="0.8825985000000001" velocity="1.0"/>
@@ -748,4 +968,59 @@
             <material name="white"/>
         </visual>
+        <collision>
+            <origin xyz="-0.055 0 0.005"/>
+            <geometry>
+                <mesh filename="file://$(find hexapod)/meshes/left_tibia.stl" scale="0.001 0.001 0.001"/>
+            </geometry>
+        </collision>
+        <xacro:inertial_box mass="0.015" x="0.01" y="0.01" z="0.01">
+            <origin xyz="-0.055 0 0.005"/>
+        </xacro:inertial_box>
+    </link>
+    <joint name="shield5_joint" type="fixed">
+        <parent link="tibia5"/>
+        <child link="shield5"/>
+        <origin xyz="0 0 0" rpy="0 0 0"/>
+    </joint>
+    <link name="shield5">
+        <visual>
+            <origin xyz="-0.055 -0.01 0"/>
+            <geometry>
+                <mesh filename="file://$(find hexapod)/meshes/shield.stl" scale="0.001 0.001 0.001"/>
+            </geometry>
+            <material name="blue"/>
+        </visual>
+        <collision>
+            <origin xyz="-0.055 -0.01 0"/>
+            <geometry>
+                <mesh filename="file://$(find hexapod)/meshes/shield.stl" scale="0.001 0.001 0.001"/>
+            </geometry>
+        </collision>
+        <xacro:inertial_box mass="0.015" x="0.01" y="0.01" z="0.01">
+            <origin xyz="-0.055 -0.01 0"/>
+        </xacro:inertial_box>
+    </link>
+    <joint name="sensor5_joint" type="fixed">
+        <parent link="tibia5"/>
+        <child link="sensor5"/>
+        <origin xyz="0 0 0" rpy="0 0 0"/>
+    </joint>
+    <link name="sensor5">
+        <visual>
+            <origin xyz="-0.0425 -0.005 -0.125"/>
+            <geometry>
+                <mesh filename="file://$(find hexapod)/meshes/micro_switch_tip.stl" scale="0.001 0.001 0.001"/>
+            </geometry>
+            <material name="white"/>
+        </visual>
+        <collision>
+            <origin xyz="-0.0425 -0.005 -0.125"/>
+            <geometry>
+                <mesh filename="file://$(find hexapod)/meshes/micro_switch_tip.stl" scale="0.001 0.001 0.001"/>
+            </geometry>
+        </collision>
+        <xacro:inertial_box mass="0.015" x="0.01" y="0.01" z="0.01">
+             <origin xyz="-0.0425 -0.005 -0.125"/>
+        </xacro:inertial_box>
     </link>
     <!-- LEG 6 (LF) -->
@@ -801,5 +1076,5 @@
         <parent link="servo12"/>
         <child link="femur6"/>
-        <origin xyz="0.045 0 0.02" rpy="${pi/2} 0 ${pi}"/>
+        <origin xyz="0.045 0 0.02" rpy="${pi/2} ${pi/4} ${pi}"/>
         <axis xyz="0 0 1" />
         <limit lower="-0.785398" upper="0.785398" effort="0.8825985000000001" velocity="1.0"/>
@@ -826,5 +1101,5 @@
         <parent link="femur6"/>
         <child link="servo18"/>
-        <origin xyz="-0.0775 0 0"/>
+        <origin xyz="-0.0775 0 0" rpy="0 0 ${pi/4}"/>
         <axis xyz="0 0 1" />
         <limit lower="-0.785398" upper="0.785398" effort="0.8825985000000001" velocity="1.0"/>
@@ -861,4 +1136,59 @@
             <material name="white"/>
         </visual>
+        <collision>
+            <origin xyz="-0.055 0 0.005"/>
+            <geometry>
+                <mesh filename="file://$(find hexapod)/meshes/left_tibia.stl" scale="0.001 0.001 0.001"/>
+            </geometry>
+        </collision>
+        <xacro:inertial_box mass="0.015" x="0.01" y="0.01" z="0.01">
+            <origin xyz="-0.055 0 0.005"/>
+        </xacro:inertial_box>
+    </link>
+    <joint name="shield6_joint" type="fixed">
+        <parent link="tibia6"/>
+        <child link="shield6"/>
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