Commit message: Gazebo URDF markers added

File: description/robot_frame.xacro (robot description, xacro)
@@ -44,4 +44,7 @@
         </xacro:inertial_box>
     </link>
+    <gazebo reference="frame">
+        <material>Gazebo/White </material>
+    </gazebo>
     <!-- FRAME SERVOS -->
     <joint name="servo1_joint" type="fixed">
@@ -68,4 +71,7 @@
         </xacro:inertial_box>
     </link>
+    <gazebo reference="servo1">
+        <material>Gazebo/Black</material>
+    </gazebo>
     <joint name="servo2_joint" type="fixed">
         <parent link="frame"/>
@@ -91,4 +97,7 @@
         </xacro:inertial_box>
     </link>
+    <gazebo reference="servo2">
+        <material>Gazebo/Black</material>
+    </gazebo>
     <joint name="servo3_joint" type="fixed">
         <parent link="frame"/>
@@ -114,4 +123,7 @@
         </xacro:inertial_box>
     </link>
+    <gazebo reference="servo3">
+        <material>Gazebo/Black</material>
+    </gazebo>
     <joint name="servo4_joint" type="fixed">
         <parent link="frame"/>
@@ -137,4 +149,7 @@
         </xacro:inertial_box>
     </link>
+    <gazebo reference="servo4">
+        <material>Gazebo/Black</material>
+    </gazebo>
     <joint name="servo5_joint" type="fixed">
         <parent link="frame"/>
@@ -160,4 +175,7 @@
         </xacro:inertial_box>
     </link>
+    <gazebo reference="servo5">
+        <material>Gazebo/Black</material>
+    </gazebo>
     <joint name="servo6_joint" type="fixed">
         <parent link="frame"/>
@@ -183,4 +201,7 @@
         </xacro:inertial_box>
     </link>
+    <gazebo reference="servo6">
+        <material>Gazebo/Black</material>
+    </gazebo>
     <!-- LEG SERVOS -->
     <!-- LEG 1 (RF) -->
@@ -210,4 +231,7 @@
         </xacro:inertial_box>
     </link>
+    <gazebo reference="coxa1">
+        <material>Gazebo/White</material>
+    </gazebo>
     <joint name="servo7_joint" type="fixed">
         <parent link="coxa1"/>
@@ -233,4 +257,7 @@
         </xacro:inertial_box>
     </link>
+    <gazebo reference="servo7">
+        <material>Gazebo/Black</material>
+    </gazebo>
     <joint name="femur1_joint" type="revolute">
         <parent link="servo7"/>
@@ -258,4 +285,7 @@
         </xacro:inertial_box>
     </link>
+    <gazebo reference="femur1">
+        <material>Gazebo/White</material>
+    </gazebo>
     <joint name="servo13_joint" type="revolute">
         <parent link="femur1"/>
@@ -283,4 +313,7 @@
         </xacro:inertial_box>
     </link>
+    <gazebo reference="servo13">
+        <material>Gazebo/Black</material>
+    </gazebo>
     <joint name="tibia1_joint" type="fixed">
         <parent link="servo13"/>
@@ -306,4 +339,7 @@
         </xacro:inertial_box>
     </link>
+    <gazebo reference="tibia1">
+        <material>Gazebo/White</material>
+    </gazebo>
     <joint name="shield1_joint" type="fixed">
         <parent link="tibia1"/>
@@ -329,4 +365,7 @@
         </xacro:inertial_box>
     </link>
+    <gazebo reference="shield1">
+        <material>Gazebo/Blue</material>
+    </gazebo>
     <joint name="sensor1_joint" type="fixed">
         <parent link="tibia1"/>
@@ -352,4 +391,7 @@
         </xacro:inertial_box>
     </link>
+    <gazebo reference="sensor1">
+        <material>Gazebo/White</material>
+    </gazebo>
     <!-- LEG 2 (RM) -->
     <joint name="coxa2_joint" type="revolute">
@@ -378,4 +420,7 @@
         </xacro:inertial_box>
     </link>
+    <gazebo reference="coxa2">
+        <material>Gazebo/White</material>
+    </gazebo>
     <joint name="servo8_joint" type="fixed">
         <parent link="coxa2"/>
@@ -401,4 +446,7 @@
         </xacro:inertial_box>
     </link>
+    <gazebo reference="servo8">
+        <material>Gazebo/Black</material>
+    </gazebo>
     <joint name="femur2_joint" type="revolute">
         <parent link="servo8"/>
@@ -426,4 +474,7 @@
         </xacro:inertial_box>
     </link>
+    <gazebo reference="femur2">
+        <material>Gazebo/White</material>
+    </gazebo>
     <joint name="servo14_joint" type="revolute">
         <parent link="femur2"/>
@@ -451,4 +502,7 @@
         </xacro:inertial_box>
     </link>
+    <gazebo reference="servo14">
+        <material>Gazebo/Black</material>
+    </gazebo>
     <joint name="tibia2_joint" type="fixed">
         <parent link="servo14"/>
@@ -474,4 +528,7 @@
         </xacro:inertial_box>
     </link>
+    <gazebo reference="tibia2">
+        <material>Gazebo/White</material>
+    </gazebo>
     <joint name="shield2_joint" type="fixed">
         <parent link="tibia2"/>
@@ -497,4 +554,7 @@
         </xacro:inertial_box>
     </link>
+    <gazebo reference="shield2">
+        <material>Gazebo/Blue</material>
+    </gazebo>
     <joint name="sensor2_joint" type="fixed">
         <parent link="tibia2"/>
@@ -520,4 +580,7 @@
         </xacro:inertial_box>
     </link>
+    <gazebo reference="sensor2">
+        <material>Gazebo/White</material>
+    </gazebo>
     <!-- LEG 3 (RB) -->
     <joint name="coxa3_joint" type="revolute">
@@ -546,4 +609,7 @@
         </xacro:inertial_box>
     </link>
+    <gazebo reference="coxa3">
+        <material>Gazebo/White</material>
+    </gazebo>
     <joint name="servo9_joint" type="fixed">
         <parent link="coxa3"/>
@@ -569,4 +635,7 @@
         </xacro:inertial_box>
     </link>
+    <gazebo reference="servo9">
+        <material>Gazebo/Black</material>
+    </gazebo>
     <joint name="femur3_joint" type="revolute">
         <parent link="servo9"/>
@@ -594,4 +663,7 @@
         </xacro:inertial_box>
     </link>
+    <gazebo reference="femur3">
+        <material>Gazebo/White</material>
+    </gazebo>
     <joint name="servo15_joint" type="revolute">
         <parent link="femur3"/>
@@ -619,4 +691,7 @@
         </xacro:inertial_box>
     </link>
+    <gazebo reference="servo15">
+        <material>Gazebo/Black</material>
+    </gazebo>
     <joint name="tibia3_joint" type="fixed">
         <parent link="servo15"/>
@@ -642,4 +717,7 @@
         </xacro:inertial_box>
     </link>
+    <gazebo reference="tibia3">
+        <material>Gazebo/White</material>
+    </gazebo>
     <joint name="shield3_joint" type="fixed">
         <parent link="tibia3"/>
@@ -665,4 +743,7 @@
         </xacro:inertial_box>
     </link>
+    <gazebo reference="shield3">
+        <material>Gazebo/Blue</material>
+    </gazebo>
     <joint name="sensor3_joint" type="fixed">
         <parent link="tibia3"/>
@@ -688,4 +769,7 @@
         </xacro:inertial_box>
     </link>
+    <gazebo reference="sensor3">
+        <material>Gazebo/White</material>
+    </gazebo>
     <!-- LEG 4 (LB) -->
     <joint name="coxa4_joint" type="revolute">
@@ -714,4 +798,7 @@
         </xacro:inertial_box>
     </link>
+    <gazebo reference="coxa4">
+        <material>Gazebo/White</material>
+    </gazebo>
     <joint name="servo10_joint" type="fixed">
         <parent link="coxa4"/>
@@ -737,4 +824,7 @@
         </xacro:inertial_box>
     </link>
+    <gazebo reference="servo10">
+        <material>Gazebo/Black</material>
+    </gazebo>
     <joint name="femur4_joint" type="revolute">
         <parent link="servo10"/>
@@ -762,4 +852,7 @@
         </xacro:inertial_box>
     </link>
+    <gazebo reference="femur4">
+        <material>Gazebo/White</material>
+    </gazebo>
     <joint name="servo16_joint" type="revolute">
         <parent link="femur4"/>
@@ -787,4 +880,7 @@
         </xacro:inertial_box>
     </link>
+    <gazebo reference="servo16">
+        <material>Gazebo/Black</material>
+    </gazebo>
     <joint name="tibia4_joint" type="fixed">
         <parent link="servo16"/>
@@ -810,4 +906,7 @@
         </xacro:inertial_box>
     </link>
+    <gazebo reference="tibia4">
+        <material>Gazebo/White</material>
+    </gazebo>
     <joint name="shield4_joint" type="fixed">
         <parent link="tibia4"/>
@@ -833,4 +932,7 @@
         </xacro:inertial_box>
     </link>
+    <gazebo reference="shield4">
+        <material>Gazebo/Blue</material>
+    </gazebo>
     <joint name="sensor4_joint" type="fixed">
         <parent link="tibia4"/>
@@ -856,4 +958,7 @@
         </xacro:inertial_box>
     </link>
+    <gazebo reference="sensor4">
+        <material>Gazebo/White</material>
+    </gazebo>
     <!-- LEG 5 (LM) -->
     <joint name="coxa5_joint" type="revolute">
@@ -882,4 +987,7 @@
         </xacro:inertial_box>
     </link>
+    <gazebo reference="coxa5">
+        <material>Gazebo/White</material>
+    </gazebo>
     <joint name="servo11_joint" type="fixed">
         <parent link="coxa5"/>
@@ -905,4 +1013,7 @@
         </xacro:inertial_box>
     </link>
+    <gazebo reference="servo11">
+        <material>Gazebo/Black</material>
+    </gazebo>
     <joint name="femur5_joint" type="revolute">
         <parent link="servo11"/>
@@ -930,4 +1041,7 @@
         </xacro:inertial_box>
     </link>
+    <gazebo reference="femur5">
+        <material>Gazebo/White</material>
+    </gazebo>
     <joint name="servo17_joint" type="revolute">
         <parent link="femur5"/>
@@ -955,4 +1069,7 @@
         </xacro:inertial_box>
     </link>
+    <gazebo reference="servo17">
+        <material>Gazebo/Black</material>
+    </gazebo>
     <joint name="tibia5_joint" type="fixed">
         <parent link="servo17"/>
@@ -978,4 +1095,7 @@
         </xacro:inertial_box>
     </link>
+    <gazebo reference="tibia5">
+        <material>Gazebo/White</material>
+    </gazebo>
     <joint name="shield5_joint" type="fixed">
         <parent link="tibia5"/>
@@ -1001,4 +1121,7 @@
         </xacro:inertial_box>
     </link>
+    <gazebo reference="shield5">
+        <material>Gazebo/Blue</material>
+    </gazebo>
     <joint name="sensor5_joint" type="fixed">
         <parent link="tibia5"/>
@@ -1024,4 +1147,7 @@
         </xacro:inertial_box>
     </link>
+    <gazebo reference="sensor5">
+        <material>Gazebo/White</material>
+    </gazebo>
     <!-- LEG 6 (LF) -->
     <joint name="coxa6_joint" type="revolute">
@@ -1050,4 +1176,7 @@
         </xacro:inertial_box>
     </link>
+    <gazebo reference="coxa6">
+        <material>Gazebo/White</material>
+    </gazebo>
     <joint name="servo12_joint" type="fixed">
         <parent link="coxa6"/>
@@ -1073,4 +1202,7 @@
         </xacro:inertial_box>
     </link>
+    <gazebo reference="servo12">
+        <material>Gazebo/Black</material>
+    </gazebo>
     <joint name="femur6_joint" type="revolute">
         <parent link="servo12"/>
@@ -1098,4 +1230,7 @@
         </xacro:inertial_box>
     </link>
+    <gazebo reference="femur6">
+        <material>Gazebo/White</material>
+    </gazebo>
     <joint name="servo18_joint" type="revolute">
         <parent link="femur6"/>
@@ -1123,4 +1258,7 @@
         </xacro:inertial_box>
     </link>
+    <gazebo reference="servo18">
+        <material>Gazebo/Black</material>
+    </gazebo>
     <joint name="tibia6_joint" type="fixed">
         <parent link="servo18"/>
@@ -1146,4 +1284,7 @@
         </xacro:inertial_box>
     </link>
+    <gazebo reference="tibia6">
+        <material>Gazebo/White</material>
+    </gazebo>
     <joint name="shield6_joint" type="fixed">
         <parent link="tibia6"/>
@@ -1169,4 +1310,7 @@
         </xacro:inertial_box>
     </link>
+    <gazebo reference="shield6">
+        <material>Gazebo/Blue</material>
+    </gazebo>
     <joint name="sensor6_joint" type="fixed">
         <parent link="tibia6"/>
@@ -1192,4 +1336,7 @@
         </xacro:inertial_box>
     </link>
+    <gazebo reference="sensor6">
+        <material>Gazebo/White</material>
+    </gazebo>
     <!-- TOP -->
     <joint name="top_cover_joint" type="fixed">
@@ -1216,4 +1363,7 @@
         </xacro:inertial_box>
     </link>
+    <gazebo reference="top_cover">
+        <material>Gazebo/Blue</material>
+    </gazebo>
     <joint name="phone_joint" type="fixed">
         <parent link="top_cover"/>
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